Commit message: robot description publisher service is added

File: deploy/ros2_nodes/go2_description/xacro/robot.xacro (robot description, xacro)
@@ -81,30 +81,4 @@
         </collision>
     </link>
-    <!--
-    <joint name="load_joint" type="fixed">
-        <parent link="trunk"/>
-        <child link="load_link"/>
-        <origin rpy="0 0 0" xyz="0 0 0"/>
-    </joint>
-    <link name="load_link">
-        <inertial>
-            <mass value="5"/>
-            <origin rpy="0 0 0" xyz="0 0 0"/>
-            <inertia ixx="0.01" ixy="0" ixz="0" iyy="0.01" iyz="0" izz="0.01"/>
-        </inertial>
-        <visual>
-            <origin rpy="0 0 0" xyz="0 0 0.2"/>
-            <geometry>
-                <box size="0.5 0.3 0.2"/>
-            </geometry>
-        </visual>
-        <collision>
-            <origin rpy="0 0 0" xyz="0 0 0"/>
-            <geometry>
-                <box size=".001 .001 .001"/>
-            </geometry>
-        </collision>
-    </link>
--->
     <xacro:leg name="FR" mirror="-1" mirror_dae= "False" front_hind="1"  front_hind_dae="True"  />
     <xacro:leg name="FL" mirror="1"  mirror_dae="True"   front_hind="1"  front_hind_dae="True"  />

Commit message: calibration parameters is added to the xacro file

File: deploy/ros2_nodes/go2_description/xacro/robot.xacro (robot description, xacro)
@@ -59,5 +59,5 @@
         <parent link="trunk"/>
         <child link="imu_link"/>
-        <origin rpy="0 0 0" xyz="0 0 0"/>
+        <origin rpy="0.001697 -0.020900 -0.000007" xyz="-0.027353 -0.005499 0.039913"/>
     </joint>
     <link name="imu_link">
@@ -81,4 +81,60 @@
         </collision>
     </link>
+    <joint name="vicon_joint" type="fixed">
+        <parent link="trunk"/>
+        <child link="vicon_link"/>
+        <origin rpy="-0.037935 -0.066371 -2.668897" xyz="0.022944 -0.000007 0.058458"/>
+    </joint>
+    <link name="vicon_link">
+        <visual>
+            <origin rpy="0 0 0" xyz="0 0 0"/>
+            <geometry>
+                <box size="0.001 0.001 0.001"/>
+            </geometry>
+            <!-- <material name="red"/> -->
+        </visual>
+    </link>
+    <joint name="infra1_joint" type="fixed">
+        <parent link="trunk"/>
+        <child link="infra1_link"/>
+        <origin rpy="-1.641669 -0.014332 -1.617155" xyz="0.321618 0.033305 0.081622"/>
+    </joint>
+    <link name="infra1_link">
+        <visual>
+            <origin rpy="0 0 0" xyz="0 0 0"/>
+            <geometry>
+                <box size="0.001 0.001 0.001"/>
+            </geometry>
+            <!-- <material name="red"/> -->
+        </visual>
+    </link>
+    <joint name="infra2_joint" type="fixed">
+        <parent link="trunk"/>
+        <child link="infra1_link"/>
+        <origin rpy="-1.640637 -0.014093 -1.611177" xyz="0.317969 -0.061919 0.082773"/>
+    </joint>
+    <link name="infra2_link">
+        <visual>
+            <origin rpy="0 0 0" xyz="0 0 0"/>
+            <geometry>
+                <box size="0.001 0.001 0.001"/>
+            </geometry>
+            <!-- <material name="red"/> -->
+        </visual>
+    </link>
+    <joint name="color_joint" type="fixed">
+        <parent link="trunk"/>
+        <child link="color_link"/>
+        <origin rpy="-1.640491 -0.011125 -1.610364" xyz="0.319415 -0.025790 0.082311"/>
+    </joint>
+    <link name="color_link">
+        <visual>
+            <origin rpy="0 0 0" xyz="0 0 0"/>
+            <geometry>
+                <box size="0.001 0.001 0.001"/>
+            </geometry>
+            <!-- <material name="red"/> -->
+        </visual>
+    </link>
     <xacro:leg name="FR" mirror="-1" mirror_dae= "False" front_hind="1"  front_hind_dae="True"  />
     <xacro:leg name="FL" mirror="1"  mirror_dae="True"   front_hind="1"  front_hind_dae="True"  />

Commit message: xacro bug fix and adding odometry publisher to the bridge

File: deploy/ros2_nodes/go2_description/xacro/robot.xacro (robot description, xacro)
@@ -111,5 +111,5 @@
     <joint name="infra2_joint" type="fixed">
         <parent link="trunk"/>
-        <child link="infra1_link"/>
+        <child link="infra2_link"/>
         <origin rpy="-1.640637 -0.014093 -1.611177" xyz="0.317969 -0.061919 0.082773"/>
     </joint>

Commit message: nav2 configurations are fixed

File: deploy/ros2_nodes/go2_description/xacro/robot.xacro (robot description, xacro)
@@ -150,4 +150,17 @@
         <axis xyz="0 0 0"/>
     </joint>
+    <link name="hesai">
+        <inertial>
+        <origin rpy="0 0 0" xyz="0 0 0"/>
+        <mass value="0"/>
+        <inertia ixx="0" ixy="0" ixz="0" iyy="0" iyz="0" izz="0"/>
+        </inertial>
+    </link>
+    <joint name="hesai_joint" type="fixed">
+        <origin rpy="0 0 1.57075" xyz="0.15 0 0.25"/>
+        <parent link="base_link"/>
+        <child link="hesai"/>
+        <axis xyz="0 0 0"/>
+    </joint>
     <xacro:leg name="FR" mirror="-1" mirror_dae= "False" front_hind="1"  front_hind_dae="True"  />
     <xacro:leg name="FL" mirror="1"  mirror_dae="True"   front_hind="1"  front_hind_dae="True"  />

Commit message: nav2 and slam toolbox configurations are fixed

File: deploy/ros2_nodes/go2_description/xacro/robot.xacro (robot description, xacro)
@@ -137,5 +137,5 @@
         </visual>
     </link>
-    <link name="utlidar">
+    <!-- <link name="utlidar">
         <inertial>
         <origin rpy="0 0 0" xyz="0 0 0"/>
@@ -149,5 +149,5 @@
         <child link="utlidar"/>
         <axis xyz="0 0 0"/>
-    </joint>
+    </joint> -->
     <link name="hesai">
         <inertial>

Commit message: navigation parameters and docker is updated

File: deploy/ros2_nodes/go2_description/xacro/robot.xacro (robot description, xacro)
@@ -137,5 +137,5 @@
         </visual>
     </link>
-    <!-- <link name="utlidar">
+    <link name="utlidar_lidar">
         <inertial>
         <origin rpy="0 0 0" xyz="0 0 0"/>
@@ -147,7 +147,7 @@
         <origin rpy="0 2.8782 0" xyz="0.28945 0 -0.046825"/>
         <parent link="base_link"/>
-        <child link="utlidar"/>
+        <child link="utlidar_lidar"/>
         <axis xyz="0 0 0"/>
-    </joint> -->
+    </joint>
     <link name="hesai">
         <inertial>
