Commit message: Isaacsim and Mujoco simulator classes are added.

File: Go2Py/assets/urdf/go2.urdf (robot description, URDF)
Before this commit: robot go2_description, 29 links, 28 joints
Links:
- removed link base
- removed link imu
- added link base_link, mass 6.921; collision box size=0.3762 0.0935 0.154; visual mesh filename=../dae/base.dae
- added link imu_link, mass 0
Joints:
- joint FL_hip_joint: parent base -> base_link
- joint FR_hip_joint: parent base -> base_link
- joint Head_upper_joint: parent base -> base_link
- joint RL_hip_joint: parent base -> base_link
- joint RR_hip_joint: parent base -> base_link
- joint imu_joint: child imu -> imu_link; parent base -> base_link
- joint radar_joint: parent base -> base_link

Commit message: sensors added to the assets urdf

File: Go2Py/assets/urdf/go2.urdf (robot description, URDF)
Before this commit: robot go2, 29 links, 28 joints
Joints:
- joint imu_joint: origin xyz=-0.02557 0 0.04232 rpy=0 0 0 -> xyz=-0.027353 -0.005499 0.039913 rpy=0.001697 -0.020900 -0.000007

File: deploy/ros2_nodes/go2_description/xacro/robot.xacro (robot description, xacro)
@@ -137,4 +137,17 @@
         </visual>
     </link>
+    <link name="utlidar">
+        <inertial>
+        <origin rpy="0 0 0" xyz="0 0 0"/>
+        <mass value="0"/>
+        <inertia ixx="0" ixy="0" ixz="0" iyy="0" iyz="0" izz="0"/>
+        </inertial>
+    </link>
+    <joint name="utlidar_joint" type="fixed">
+        <origin rpy="0 2.8782 0" xyz="0.28945 0 -0.046825"/>
+        <parent link="base_link"/>
+        <child link="utlidar"/>
+        <axis xyz="0 0 0"/>
+    </joint>
     <xacro:leg name="FR" mirror="-1" mirror_dae= "False" front_hind="1"  front_hind_dae="True"  />
     <xacro:leg name="FL" mirror="1"  mirror_dae="True"   front_hind="1"  front_hind_dae="True"  />

Commit message: utlidar extrinsics updated

File: Go2Py/assets/urdf/go2.urdf (robot description, URDF)
Before this commit: robot go2, 29 links, 28 joints
Links:
- removed link radar
- added link color_link; visual box size=0.001 0.001 0.001
- added link infra1_link; visual box size=0.001 0.001 0.001
- added link infra2_link; visual box size=0.001 0.001 0.001
- added link utlidar, mass 0
- added link vicon_link; visual box size=0.001 0.001 0.001
Joints:
- removed joint radar_joint
- added joint color_joint: type fixed, parent trunk, child color_link, origin xyz=0.319415 -0.025790 0.082311 rpy=-1.640491 -0.011125 -1.610364
- added joint infra1_joint: type fixed, parent trunk, child infra1_link, origin xyz=0.321618 0.033305 0.081622 rpy=-1.641669 -0.014332 -1.617155
- added joint infra2_joint: type fixed, parent trunk, child infra1_link, origin xyz=0.317969 -0.061919 0.082773 rpy=-1.640637 -0.014093 -1.611177
- added joint utlidar_joint: type fixed, parent base_link, child utlidar, origin xyz=0.28945 0 -0.046825 rpy=0 2.8782 0, axis 0 0 0
- added joint vicon_joint: type fixed, parent trunk, child vicon_link, origin xyz=0.022944 -0.000007 0.058458 rpy=-0.037935 -0.066371 -2.668897

Commit message: Go2 URDF bug is fixed

File: Go2Py/assets/urdf/go2.urdf (robot description, URDF)
Before this commit: robot go2, 33 links, 32 joints
Joints:
- joint color_joint: parent trunk -> base_link
- joint infra1_joint: parent trunk -> base_link
- joint infra2_joint: parent trunk -> base_link
- joint vicon_joint: parent trunk -> base_link

Commit message: Many modifs.

File: Go2Py/assets/urdf/go2.urdf (robot description, URDF)
Before this commit: robot go2, 33 links, 32 joints
Links:
- removed link color_link
- removed link infra1_link
- removed link infra2_link
- removed link vicon_link
Joints:
- removed joint color_joint
- removed joint infra1_joint
- removed joint infra2_joint
- removed joint vicon_joint

Commit message: go2 with arm and mpc example added.

File: Go2Py/assets/urdf/go2.urdf (robot description, URDF)
Before this commit: robot go2, 29 links, 28 joints
Links:
- link FL_calf: geometry collision cylinder length=0.12 radius=0.012; visual mesh filename=../go2_assets/dae/calf.dae
- link FL_foot: geometry collision sphere radius=0.022; visual mesh filename=../go2_assets/dae/foot.dae
- link FL_hip: geometry visual mesh filename=../go2_assets/dae/hip.dae
- link FL_thigh: geometry collision box size=0.213 0.0245 0.034; visual mesh filename=../go2_assets/dae/thigh.dae
- link FR_calf: geometry collision cylinder length=0.12 radius=0.013; visual mesh filename=../go2_assets/dae/calf_mirror.dae
- link FR_foot: geometry collision sphere radius=0.022; visual mesh filename=../go2_assets/dae/foot.dae
- link FR_hip: geometry visual mesh filename=../go2_assets/dae/hip.dae
- link FR_thigh: geometry collision box size=0.213 0.0245 0.034; visual mesh filename=../go2_assets/dae/thigh_mirror.dae
- link RL_calf: geometry collision cylinder length=0.12 radius=0.013; visual mesh filename=../go2_assets/dae/calf.dae
- link RL_foot: geometry collision sphere radius=0.022; visual mesh filename=../go2_assets/dae/foot.dae
- link RL_hip: geometry visual mesh filename=../go2_assets/dae/hip.dae
- link RL_thigh: geometry collision box size=0.213 0.0245 0.034; visual mesh filename=../go2_assets/dae/thigh.dae
- link RR_calf: geometry collision cylinder length=0.12 radius=0.013; visual mesh filename=../go2_assets/dae/calf_mirror.dae
- link RR_foot: geometry collision sphere radius=0.022; visual mesh filename=../go2_assets/dae/foot.dae
- link RR_hip: geometry visual mesh filename=../go2_assets/dae/hip.dae
- link RR_thigh: geometry collision box size=0.213 0.0245 0.034; visual mesh filename=../go2_assets/dae/thigh_mirror.dae
- link base_link: geometry collision box size=0.3762 0.0935 0.154; visual mesh filename=../go2_assets/dae/base.dae
